File: schematics/ebow/ebow.kicad_sch (KiCad schematic)
At the start: 11 parts, among them U1 LM386

Commit message: first round no routing for pcb
Parts:
- added BT1: Battery, audiostuff:battery_connector_9v, symbol Device:Battery
- added FID1, FID2: Fiducial, Fiducial:Fiducial_0.5mm_Mask1.5mm, symbol Mechanical:Fiducial
- added H1, H2: MountingHole, MountingHole:MountingHole_2.1mm, symbol Mechanical:MountingHole
- added SW1: SW_SPDT, audiostuff:switch-2-mode, symbol Switch:SW_SPDT
- L1: footprint Capacitor_SMD:C_0201_0603Metric -> audiostuff:Inductor
- L2: footprint (none) -> audiostuff:Inductor
- U1: footprint (none) -> audiostuff:lm386-smd
Connections:
- net +9V: now also BT1.1 (+), SW1.1 (A); no longer R4.2, U1.6 (V+)
- net GND: now also BT1.2 (-)
- new net: R4.2, SW1.2 (B), U1.6 (V+)
Other:
- moved on the sheet: C1, C2, C3, C4, C5, D1, L1, L2, R1, R4, U1

Commit message: more edits
Connections:
- net GND: now also L1.2; no longer L1.1
- net at C2.1, C3.1, R1.1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: now also L1.1; no longer L1.2
Other:
- moved on the sheet: L1
Changed lines of the file:
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@@
 	(symbol
 		(lib_id "Device:L")
-		(at 45.72 113.03 90)
+		(at 45.72 113.03 270)
 		(unit 1)
 		(exclude_from_sim no)

Commit message: corrections
Parts:
- added FID3: Fiducial, Fiducial:Fiducial_0.5mm_Mask1.5mm, symbol Mechanical:Fiducial
- R1, R4: footprint Resistor_SMD:R_0201_0603Metric -> Resistor_SMD:R_0201_0603Metric_Pad0.64x0.40mm_HandSolder
Changed lines of the file:
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@@
 (kicad_sch
-	(version 20231120)
+	(version 20250114)
 	(generator "eeschema")
-	(generator_version "8.0")
+	(generator_version "9.0")
 	(paper "A4")
 	(title_block
@@
 	)
 	(symbol
+		(lib_id "Mechanical:Fiducial")
+		(at 247.65 91.44 0)
+		(unit 1)
+		(exclude_from_sim yes)
+		(in_bom no)
+		(on_board yes)
+		(dnp no)
+		(fields_autoplaced yes)
+		(property "Reference" "FID3"
+			(at 250.19 90.1699 0)
+			(effects
+				(font
+					(size 1.27 1.27)
+				)
+				(justify left)
+			)
+		)
+		(property "Value" "Fiducial"
+			(at 250.19 92.7099 0)
+			(effects
+				(font
+					(size 1.27 1.27)
+				)
+				(justify left)
+			)
+		)
+		(property "Footprint" "Fiducial:Fiducial_0.5mm_Mask1.5mm"
+			(at 247.65 91.44 0)
+			(effects
+				(font
+					(size 1.27 1.27)
+				)
+				(hide yes)
+			)
+		)
+		(property "Datasheet" "~"
+			(at 247.65 91.44 0)
+			(effects
+				(font
+					(size 1.27 1.27)
+				)
+				(hide yes)
+			)
+		)
+		(property "Description" "Fiducial Marker"
+			(at 247.65 91.44 0)
+			(effects
+				(font
+					(size 1.27 1.27)
+				)
+				(hide yes)
+			)
+		)
+		(instances
+			(project "ebow"
+				(path "/e1b4dd4e-8d19-49ab-849b-d4c53e40bae1"
+					(reference "FID3")
+					(unit 1)
+				)
+			)
+		)
+	)
+	(symbol
 		(lib_id "Device:R")
 		(at 54.61 128.27 0)
@@
 			)
 		)
-		(property "Footprint" "Resistor_SMD:R_0201_0603Metric"
+		(property "Footprint" "Resistor_SMD:R_0201_0603Metric_Pad0.64x0.40mm_HandSolder"
 			(at 52.832 128.27 90)
 			(effects
@@
 					(size 1.27 1.27)
 				)
-			)
-		)
-		(property "Footprint" "Resistor_SMD:R_0201_0603Metric"
+				(hide yes)
+			)
+		)
+		(property "Footprint" "Resistor_SMD:R_0201_0603Metric_Pad0.64x0.40mm_HandSolder"
 			(at 146.558 109.22 90)
 			(effects
@@
 		)
 	)
+	(embedded_fonts no)
 )
